File: hw/sch_pcb/TFASPDIMU01B.kicad_pcb (KiCad board)
At the start: 2 copper layers, 36 x 14 mm, 26 parts, among them J1 SM07B-GHS-TB, U1 SDP3x, U2 ICM-20948, U4 MIC5504-3.3YM5-TR, U5 MIC5504-1.8YM5-TR, U6 TXS0108EPW

Commit message: Edit schema
Parts:
- added U3: TCA9617A, Package_SO:TSSOP-8_3x3mm_P0.65mm, F.Cu at (186.8, 112.9)
Changed lines of the file:
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@@
   (net 34 "unconnected-(U6-Pad9)")
   (net 35 "unconnected-(U6-Pad12)")
+  (net 36 "unconnected-(U3-Pad1)")
+  (net 37 "unconnected-(U3-Pad2)")
+  (net 38 "unconnected-(U3-Pad3)")
+  (net 39 "unconnected-(U3-Pad4)")
+  (net 40 "unconnected-(U3-Pad5)")
+  (net 41 "unconnected-(U3-Pad6)")
+  (net 42 "unconnected-(U3-Pad7)")
+  (net 43 "unconnected-(U3-Pad8)")
   (footprint "Mlab_R:SMD-0603" (layer "F.Cu")
     (at 152.6525 99.08 90)
@@
       (offset (xyz 0 0 0))
       (scale (xyz 1 1 1))
+      (rotate (xyz 0 0 0))
+    )
+  )
+  (footprint "Package_SO:TSSOP-8_3x3mm_P0.65mm" (layer "F.Cu")
+    (at 186.817 112.903)
+    (descr "TSSOP8: plastic thin shrink small outline package; 8 leads; body width 3 mm; (see NXP SSOP-TSSOP-VSO-REFLOW.pdf and sot505-1_po.pdf)")
+    (tags "SSOP 0.65")
+    (property "Sheetfile" "TFASPDIMU01B.kicad_sch")
+    (property "Sheetname" "")
+    (attr smd)
+    (fp_text reference "U3" (at 0 -2.55) (layer "F.SilkS")
+      (effects (font (size 1 1) (thickness 0.15)))
+    )
+    (fp_text value "TCA9617A" (at 0 2.55) (layer "F.Fab")
+      (effects (font (size 1 1) (thickness 0.15)))
+    )
+    (fp_text user "${REFERENCE}" (at 0 0) (layer "F.Fab")
+      (effects (font (size 0.6 0.6) (thickness 0.15)))
+    )
+    (fp_line (start -1.625 -1.5) (end -2.7 -1.5) (layer "F.SilkS") (width 0.15))
+    (fp_line (start -1.625 -1.625) (end -1.625 -1.5) (layer "F.SilkS") (width 0.15))
+    (fp_line (start -1.625 1.625) (end -1.625 1.4) (layer "F.SilkS") (width 0.15))
+    (fp_line (start 1.625 1.625) (end 1.625 1.4) (layer "F.SilkS") (width 0.15))
+    (fp_line (start -1.625 -1.625) (end 1.625 -1.625) (layer "F.SilkS") (width 0.15))
+    (fp_line (start 1.625 -1.625) (end 1.625 -1.4) (layer "F.SilkS") (width 0.15))
+    (fp_line (start -1.625 1.625) (end 1.625 1.625) (layer "F.SilkS") (width 0.15))
+    (fp_line (start -2.95 1.8) (end 2.95 1.8) (layer "F.CrtYd") (width 0.05))
+    (fp_line (start 2.95 -1.8) (end 2.95 1.8) (layer "F.CrtYd") (width 0.05))
+    (fp_line (start -2.95 -1.8) (end -2.95 1.8) (layer "F.CrtYd") (width 0.05))
+    (fp_line (start -2.95 -1.8) (end 2.95 -1.8) (layer "F.CrtYd") (width 0.05))
+    (fp_line (start 1.5 1.5) (end -1.5 1.5) (layer "F.Fab") (width 0.15))
+    (fp_line (start 1.5 -1.5) (end 1.5 1.5) (layer "F.Fab") (width 0.15))
+    (fp_line (start -0.5 -1.5) (end 1.5 -1.5) (layer "F.Fab") (width 0.15))
+    (fp_line (start -1.5 1.5) (end -1.5 -0.5) (layer "F.Fab") (width 0.15))
+    (fp_line (start -1.5 -0.5) (end -0.5 -1.5) (layer "F.Fab") (width 0.15))
+    (pad "1" smd rect locked (at -2.15 -0.975) (size 1.1 0.4) (layers "F.Cu" "F.Paste" "F.Mask")
+      (net 36 "unconnected-(U3-Pad1)") (pinfunction "VCCA") (pintype "power_in"))
+    (pad "2" smd rect locked (at -2.15 -0.325) (size 1.1 0.4) (layers "F.Cu" "F.Paste" "F.Mask")
+      (net 37 "unconnected-(U3-Pad2)") (pinfunction "SCLA") (pintype "bidirectional"))
+    (pad "3" smd rect locked (at -2.15 0.325) (size 1.1 0.4) (layers "F.Cu" "F.Paste" "F.Mask")
+      (net 38 "unconnected-(U3-Pad3)") (pinfunction "SDAA") (pintype "bidirectional"))
+    (pad "4" smd rect locked (at -2.15 0.975) (size 1.1 0.4) (layers "F.Cu" "F.Paste" "F.Mask")
+      (net 39 "unconnected-(U3-Pad4)") (pinfunction "GND") (pintype "power_in"))
+    (pad "5" smd rect locked (at 2.15 0.975) (size 1.1 0.4) (layers "F.Cu" "F.Paste" "F.Mask")
+      (net 40 "unconnected-(U3-Pad5)") (pinfunction "EN") (pintype "input"))
+    (pad "6" smd rect locked (at 2.15 0.325) (size 1.1 0.4) (layers "F.Cu" "F.Paste" "F.Mask")
+      (net 41 "unconnected-(U3-Pad6)") (pinfunction "SDAB") (pintype "bidirectional"))
+    (pad "7" smd rect locked (at 2.15 -0.325) (size 1.1 0.4) (layers "F.Cu" "F.Paste" "F.Mask")
+      (net 42 "unconnected-(U3-Pad7)") (pinfunction "SCLB") (pintype "bidirectional"))
+    (pad "8" smd rect locked (at 2.15 -0.975) (size 1.1 0.4) (layers "F.Cu" "F.Paste" "F.Mask")
+      (net 43 "unconnected-(U3-Pad8)") (pinfunction "VCCB") (pintype "power_in"))
+    (model "${KISYS3DMOD}/Package_SO.3dshapes/TSSOP-8_3x3mm_P0.65mm.wrl"
+      (offset (xyz 0 0 0))
+      (scale (xyz 1 1 1))
