File: hw/sch_pcb/TFASPDIMU02A.kicad_sch (KiCad schematic)
At the start: 38 parts, among them J1 SM04B-GHS-TB, M1 HOLE_TF, M2 HOLE_TF, M3 HOLE_TF, M7 HOLE_TF, U1 SDP3x, U2 ICM-20948, U3 TCA9617A, U4 MIC5504-3.3YM5-TR, U5 MIC5504-1.8YM5-TR, U6 TCA9617A

Commit message: Edit bom
Parts:
- C1, C10, C12, C13, C2, C3, C4, C9: UST_ID 5c70984712875079b91f8b4c -> 5c70984812875079b91f8bdb
- C11: UST_ID 5c70984812875079b91f8bbd -> 610d01671287500165a97012
- C5, C6, C7, C8: UST_ID 5c70984712875079b91f8b50 -> 610cff5e1287500165a96ff9
- R1, R11: UST_ID (none) -> 610d02e21287500165a97051
- R10, R2, R3: UST_ID (none) -> 610d02801287500165a9703c
- R4, R5, R6, R7, R8, R9: UST_ID (none) -> 5c70984512875079b91f894c
- U1: UST_ID 5c70984812875079b91f8bd0 -> 5e32e1111287502a337d0b08
- U3, U6: UST_ID (none) -> 610d03ad1287500165a97076
Changed lines of the file:
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@@
       (effects (font (size 1.27 1.27)) hide)
     )
-    (property "UST_ID" "" (id 4) (at 90.805 141.605 0)
+    (property "UST_ID" "5c70984512875079b91f894c" (id 4) (at 90.805 141.605 0)
       (effects (font (size 1.27 1.27)) hide)
     )
@@
       (effects (font (size 1.27 1.27)) hide)
     )
-    (property "UST_ID" "" (id 4) (at 97.155 141.605 0)
+    (property "UST_ID" "5c70984512875079b91f894c" (id 4) (at 97.155 141.605 0)
       (effects (font (size 1.27 1.27)) hide)
     )
@@
       (effects (font (size 1.27 1.27)) hide)
     )
-    (property "UST_ID" "" (id 4) (at 128.27 102.87 0)
+    (property "UST_ID" "5c70984512875079b91f894c" (id 4) (at 128.27 102.87 0)
       (effects (font (size 1.27 1.27)) hide)
     )
@@
       (effects (font (size 1.27 1.27)) hide)
     )
-    (property "UST_ID" "" (id 4) (at 134.62 102.87 0)
+    (property "UST_ID" "5c70984512875079b91f894c" (id 4) (at 134.62 102.87 0)
       (effects (font (size 1.27 1.27)) hide)
     )
@@
       (effects (font (size 1.27 1.27)) hide)
     )
-    (property "UST_ID" "" (id 4) (at 159.385 35.56 0)
+    (property "UST_ID" "5c70984512875079b91f894c" (id 4) (at 159.385 35.56 0)
       (effects (font (size 1.27 1.27)) hide)
     )
@@
       (effects (font (size 1.27 1.27)) hide)
     )
-    (property "UST_ID" "" (id 4) (at 165.735 35.56 0)
+    (property "UST_ID" "5c70984512875079b91f894c" (id 4) (at 165.735 35.56 0)
       (effects (font (size 1.27 1.27)) hide)
     )
@@
       (effects (font (size 1.27 1.27)) hide)
     )
+    (property "UST_ID" "610d02e21287500165a97051" (id 4) (at 181.61 113.03 0)
+      (effects (font (size 1.27 1.27)) hide)
+    )
     (pin "1")
     (pin "2")
@@
       (effects (font (size 1.27 1.27)) hide)
     )
+    (property "UST_ID" "610d02e21287500165a97051" (id 4) (at 181.61 115.57 0)
+      (effects (font (size 1.27 1.27)) hide)
+    )
     (pin "1")
     (pin "2")
@@
       (effects (font (size 1.27 1.27)) hide)
     )
-    (property "UST_ID" "" (id 4) (at 191.77 102.87 0)
+    (property "UST_ID" "610d02801287500165a9703c" (id 4) (at 191.77 102.87 0)
       (effects (font (size 1.27 1.27)) hide)
     )
@@
       (effects (font (size 1.27 1.27)) hide)
     )
-    (property "UST_ID" "" (id 4) (at 198.12 102.87 0)
+    (property "UST_ID" "610d02801287500165a9703c" (id 4) (at 198.12 102.87 0)
       (effects (font (size 1.27 1.27)) hide)
     )
@@
       (effects (font (size 1.27 1.27)) hide)
     )
+    (property "UST_ID" "610d02801287500165a9703c" (id 4) (at 217.17 55.88 0)
+      (effects (font (size 1.27 1.27)) hide)
+    )
     (pin "1")
     (pin "2")
@@
       (effects (font (size 1.27 1.27)) hide)
     )
-    (property "UST_ID" "5c70984812875079b91f8bbd" (id 4) (at 22.86 75.565 0)
+    (property "UST_ID" "610d01671287500165a97012" (id 4) (at 22.86 75.565 0)
       (effects (font (size 1.27 1.27)) hide)
     )
@@
       (effects (font (size 1.27 1.27)) hide)
     )
-    (property "UST_ID" "5c70984712875079b91f8b4c" (id 4) (at 59.055 127.635 0)
+    (property "UST_ID" "5c70984812875079b91f8bdb" (id 4) (at 59.055 127.635 0)
       (effects (font (size 1.27 1.27)) hide)
     )
@@
       (effects (font (size 1.27 1.27)) hide)
     )
-    (property "UST_ID" "5c70984712875079b91f8b4c" (id 4) (at 79.375 127.635 0)
+    (property "UST_ID" "5c70984812875079b91f8bdb" (id 4) (at 79.375 127.635 0)
       (effects (font (size 1.27 1.27)) hide)
     )
@@
       (effects (font (size 1.27 1.27)) hide)
     )
-    (property "UST_ID" "5c70984712875079b91f8b4c" (id 4) (at 88.265 164.465 0)
+    (property "UST_ID" "5c70984812875079b91f8bdb" (id 4) (at 88.265 164.465 0)
       (effects (font (size 1.27 1.27)) hide)
     )
@@
       (effects (font (size 1.27 1.27)) hide)
     )
-    (property "UST_ID" "5c70984712875079b91f8b4c" (id 4) (at 120.015 31.75 0)
+    (property "UST_ID" "5c70984812875079b91f8bdb" (id 4) (at 120.015 31.75 0)
       (effects (font (size 1.27 1.27)) hide)
     )
@@
       (effects (font (size 1.27 1.27)) hide)
     )
-    (property "UST_ID" "5c70984712875079b91f8b4c" (id 4) (at 146.685 31.75 0)
+    (property "UST_ID" "5c70984812875079b91f8bdb" (id 4) (at 146.685 31.75 0)
       (effects (font (size 1.27 1.27)) hide)
     )
@@
       (effects (font (size 1.27 1.27)) hide)
     )
-    (property "UST_ID" "5c70984712875079b91f8b4c" (id 4) (at 149.86 99.06 0)
+    (property "UST_ID" "5c70984812875079b91f8bdb" (id 4) (at 149.86 99.06 0)
       (effects (font (size 1.27 1.27)) hide)
     )
@@
       (effects (font (size 1.27 1.27)) hide)
     )
-    (property "UST_ID" "5c70984712875079b91f8b4c" (id 4) (at 176.53 99.06 0)
+    (property "UST_ID" "5c70984812875079b91f8bdb" (id 4) (at 176.53 99.06 0)
       (effects (font (size 1.27 1.27)) hide)
     )
@@
       (effects (font (size 1.27 1.27)) hide)
     )
-    (property "UST_ID" "5c70984712875079b91f8b4c" (id 4) (at 197.485 33.02 0)
+    (property "UST_ID" "5c70984812875079b91f8bdb" (id 4) (at 197.485 33.02 0)
       (effects (font (size 1.27 1.27)) hide)
     )
@@
       (effects (font (size 1.27 1.27)) hide)
     )
-    (property "UST_ID" "5c70984712875079b91f8b50" (id 4) (at 234.315 118.11 0)
+    (property "UST_ID" "610cff5e1287500165a96ff9" (id 4) (at 234.315 118.11 0)
       (effects (font (size 1.27 1.27)) hide)
     )
@@
       (effects (font (size 1.27 1.27)) hide)
     )
-    (property "UST_ID" "5c70984712875079b91f8b50" (id 4) (at 234.315 148.59 0)
+    (property "UST_ID" "610cff5e1287500165a96ff9" (id 4) (at 234.315 148.59 0)
       (effects (font (size 1.27 1.27)) hide)
     )
@@
       (effects (font (size 1.27 1.27)) hide)
     )
-    (property "UST_ID" "5c70984712875079b91f8b50" (id 4) (at 271.145 118.11 0)
+    (property "UST_ID" "610cff5e1287500165a96ff9" (id 4) (at 271.145 118.11 0)
       (effects (font (size 1.27 1.27)) hide)
     )
@@
       (effects (font (size 1.27 1.27)) hide)
     )
-    (property "UST_ID" "5c70984712875079b91f8b50" (id 4) (at 271.145 148.59 0)
+    (property "UST_ID" "610cff5e1287500165a96ff9" (id 4) (at 271.145 148.59 0)
       (effects (font (size 1.27 1.27)) hide)
     )
@@
       (effects (font (size 1.524 1.524)) hide)
     )
-    (property "UST_ID" "5c70984812875079b91f8bd0" (id 4) (at 180.975 53.34 0)
+    (property "UST_ID" "5e32e1111287502a337d0b08" (id 4) (at 180.975 53.34 0)
       (effects (font (size 1.27 1.27)) hide)
     )
@@
       (effects (font (size 1.27 1.27)) hide)
     )
+    (property "UST_ID" "610d03ad1287500165a97076" (id 4) (at 135.255 48.26 0)
+      (effects (font (size 1.27 1.27)) hide)
+    )
     (pin "1")
     (pin "2")
@@
       (effects (font (size 1.27 1.27)) hide)
     )
+    (property "UST_ID" "610d03ad1287500165a97076" (id 4) (at 165.1 115.57 0)
+      (effects (font (size 1.27 1.27)) hide)
+    )
